File: RTFMJoy.kicad_pcb (KiCad board)
At the start: 2 copper layers, 22 parts, among them J1 Conn_02x05_Top_Bottom, J2 Conn_02x05_Top_Bottom, U1 74LS240, U2 74LS240, U3 74LS139

Commit message: Add files via upload
Corrected an issue where the enable pins from U3 were connected to the wrong 74LS240
Connections:
- U3 pad 5: Net-(U2-Pad1) -> Net-(U1-Pad1)
- U3 pad 6: Net-(U1-Pad1) -> Net-(U2-Pad1)
Routing:
- net GND: track 213.3 -> 221.2 mm
- net Net-(U1-Pad1): track 59.9 -> 57.3 mm
Other:
- board outline added: 49 x 69 mm
- board text added: "Use resistors -OR- resistor array, not both"
