File: RTFMJoy.sch (KiCad schematic (older format))
At the start: 22 parts, among them J1 Conn_02x05_Top_Bottom, J2 Conn_02x05_Top_Bottom, U1 74LS240, U2 74LS240, U3 74LS139

Commit message: Add files via upload
Corrected an issue where the enable pins from U3 were connected to the wrong 74LS240
Connections:
- net at U1.1 (OEa), U1.19 (OEb): now also U3.5 (~Q1); no longer U3.6 (~Q2)
- net at U2.1 (OEa), U2.19 (OEb): now also U3.6 (~Q2); no longer U3.5 (~Q1)
Changed lines of the file:
@@
 	4650 2850 4650 2950
 Wire Wire Line
-	4650 2950 4650 4300
+	4650 2950 4650 4100
 Connection ~ 4650 2950
 Wire Wire Line
@@
 NoConn ~ 9400 5050
 Wire Wire Line
-	9400 4100 7150 4100
-Wire Wire Line
-	7150 2950 7150 4100
-Wire Wire Line
 	7750 5000 9300 5000
 Wire Wire Line
@@
 Text Notes 1800 4850 0    50   ~ 0
 OPTIONAL: Use resistor network or individual resistors.
-Wire Wire Line
-	4650 4300 9400 4300
 Text Notes 5250 6450 0    50   ~ 0
 OPTIONAL: Use resistor network or individual resistors.
@@
 Wire Wire Line
 	6850 950  7300 950
+Wire Wire Line
+	9400 4300 7150 4300
+Wire Wire Line
+	7150 2950 7150 4300
+Wire Wire Line
+	9400 4100 4650 4100
 $EndSCHEMATC
